Commit message: Add monopod-mesh robot

File: urdf/monopod_mesh.urdf (robot description, URDF)
Before this commit: robot object, 4 links, 3 joints
Links:
- removed link l_rigid_leg
- link base_link: geometry collision mesh filename=package://monopod_description/meshes/monopod_base.dae; visual mesh filename=package://monopod_description/meshes/monopod_base.dae
- link l_bounding_sphere: geometry collision sphere radius=0.399; visual sphere radius=0.399
- link l_mobile_leg: geometry collision mesh filename=package://monopod_description/meshes/monopod_leg.dae; visual mesh filename=package://monopod_description/meshes/monopod_leg.dae
Joints:
- removed joint j_rigid_leg
- joint j_mobile_leg: origin xyz=0 0 -0.245 -> xyz=0 0 -0.249
